File: kicad/ind_switch.kicad_sch (KiCad schematic)
At the start: 3 parts, among them SW2 SW_DIP_x01

Commit message: Post zip cleanups
Parts:
- D9: renamed from D11; footprint (none) -> Diode_SMD:D_0805_2012Metric
- R2: value 10k -> 680; footprint (none) -> Resistor_SMD:R_0805_2012Metric
- SW2: footprint (none) -> switch:200MSP1T1B1M2QEH

Commit message: Initial PCB layout
Parts:
- renumbered D9 to D15, SW2 to SW1
Changed lines of the file:
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@@
 		(dnp no)
 		(fields_autoplaced yes)
-		(property "Reference" "#PWR010"
+		(property "Reference" "#PWR016"
 			(at 156.21 113.03 0)
 			(effects
@@
 			(project "sk"
 				(path "/87c8109f-f49d-4ab5-a5ef-17a7399b7634/74173968-0e33-4bf5-8826-2e559819973c"
-					(reference "#PWR010")
+					(reference "#PWR016")
 					(unit 1)
 				)
 				(path "/87c8109f-f49d-4ab5-a5ef-17a7399b7634/7be091f9-37cf-4a27-ad84-5117883f8787"
-					(reference "#PWR09")
+					(reference "#PWR015")
 					(unit 1)
 				)
 				(path "/87c8109f-f49d-4ab5-a5ef-17a7399b7634/fd790dce-4c78-46a3-8875-ecdd4bb23b82"
-					(reference "#PWR011")
+					(reference "#PWR017")
 					(unit 1)
 				)
 				(path "/87c8109f-f49d-4ab5-a5ef-17a7399b7634/2ddfa9ed-3b29-4ef0-a3a1-0c86e22b1205"
-					(reference "#PWR012")
+					(reference "#PWR018")
 					(unit 1)
 				)
 				(path "/87c8109f-f49d-4ab5-a5ef-17a7399b7634/9382501c-2438-47d9-ac28-37d798e8ff98"
-					(reference "#PWR013")
+					(reference "#PWR019")
 					(unit 1)
 				)
 				(path "/87c8109f-f49d-4ab5-a5ef-17a7399b7634/674cd22f-ee88-40ad-a5b6-2ca2aadec3d2"
-					(reference "#PWR014")
+					(reference "#PWR020")
 					(unit 1)
 				)
@@
 		(dnp no)
 		(fields_autoplaced yes)
-		(property "Reference" "D9"
+		(property "Reference" "D15"
 			(at 158.75 100.0124 90)
 			(effects
@@
 			(project "sk"
 				(path "/87c8109f-f49d-4ab5-a5ef-17a7399b7634/74173968-0e33-4bf5-8826-2e559819973c"
-					(reference "D9")
+					(reference "D15")
 					(unit 1)
 				)
 				(path "/87c8109f-f49d-4ab5-a5ef-17a7399b7634/7be091f9-37cf-4a27-ad84-5117883f8787"
-					(reference "D8")
+					(reference "D14")
 					(unit 1)
 				)
 				(path "/87c8109f-f49d-4ab5-a5ef-17a7399b7634/fd790dce-4c78-46a3-8875-ecdd4bb23b82"
-					(reference "D10")
+					(reference "D16")
 					(unit 1)
 				)
 				(path "/87c8109f-f49d-4ab5-a5ef-17a7399b7634/2ddfa9ed-3b29-4ef0-a3a1-0c86e22b1205"
-					(reference "D11")
+					(reference "D17")
 					(unit 1)
 				)
 				(path "/87c8109f-f49d-4ab5-a5ef-17a7399b7634/9382501c-2438-47d9-ac28-37d798e8ff98"
-					(reference "D12")
+					(reference "D18")
 					(unit 1)
 				)
 				(path "/87c8109f-f49d-4ab5-a5ef-17a7399b7634/674cd22f-ee88-40ad-a5b6-2ca2aadec3d2"
-					(reference "D13")
+					(reference "D19")
 					(unit 1)
 				)
@@
 		(dnp no)
 		(fields_autoplaced yes)
-		(property "Reference" "SW2"
+		(property "Reference" "SW1"
 			(at 146.05 83.82 0)
 			(effects
@@
 			(project "sk"
 				(path "/87c8109f-f49d-4ab5-a5ef-17a7399b7634/74173968-0e33-4bf5-8826-2e559819973c"
+					(reference "SW1")
+					(unit 1)
+				)
+				(path "/87c8109f-f49d-4ab5-a5ef-17a7399b7634/7be091f9-37cf-4a27-ad84-5117883f8787"
 					(reference "SW2")
 					(unit 1)
 				)
-				(path "/87c8109f-f49d-4ab5-a5ef-17a7399b7634/7be091f9-37cf-4a27-ad84-5117883f8787"
-					(reference "SW1")
-					(unit 1)
-				)
