File: kicad/psu_230vac.kicad_sch (KiCad schematic)
At the start: 14 parts, among them T1 FP12-3800

Commit message: Post zip cleanups
Parts:
- removed C1: 2.2m, symbol Device:C_Polarized
- removed C6, C7: 100n, symbol Device:C
- removed FL1: Filter_EMI_CLC, symbol Device:Filter_EMI_CLC
- removed L1: 47u, 69 mOhms, symbol Device:L
- added FL2: SBSGP5000472MXT, emif:SBSGP5000472MXT, symbol SBSGP5000472MXT:SBSGP5000472MXT
- C1: renamed from C2; value 2.2m -> 4.7m; footprint (none) -> cap-4700u:CAPPRD1000W80D2200H3700
- C2: renamed from C3; value 2.2m -> 4.7m; footprint (none) -> cap-4700u:CAPPRD1000W80D2200H3700
- C3: renamed from C4; value 220u -> 2.2m; footprint (none) -> cap-2200u:CAPPRD750W80D1600H3800
- C4: renamed from C5; value 220u -> 2.2m; footprint (none) -> cap-2200u:CAPPRD750W80D1600H3800
- D1: value GBU4A -> B25C5000
- F2: footprint (none) -> polyfuse:FUSC7451X180N
- T1: value FP12-3800 -> FP10-4800; footprint FP12-3800:XFMR_FP12-3800 -> fp10-4800:XFMR_FP10-4800
Connections:
- net +12VDC: now also F2.2
- net NEUTRAL: now also FL2.2
- net at F1.2: now also FL2.1
- net at T1.1: now also FL2.3
- net at D1.3, T1.5, T1.8: no longer D1.2, T1.6, T1.7
- new net: D1.2, T1.6, T1.7
Other:
- moved on the sheet: C1, C2, C3, C4, F1

Commit message: Initial PCB layout
Parts:
- F1: footprint (none) -> fuse:FUSC6125X279N
- RV1: footprint (none) -> varistor:VARC8250X200N
- renumbered FL2 to FL1
Connections:
- net NEUTRAL: now also FL1.3; no longer FL1.2
- net DOUT+: now reaches D1.1 (+), F2.1
- net at T1.1: now also FL1.2; no longer FL1.3
- net TOUT+: now reaches D1.3, T1.5, T1.8
- net TOUT-: now reaches D1.2, T1.6, T1.7
Other:
- moved on the sheet: C1, C2, C3, C4, F2

Commit message: Post review
Other:
- note added: "Sprawdzić opór bezpiecznika resetowalnego"
- note added: "Warystor przed bezpiecznikiem?"
Changed lines of the file:
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@@
+		)
+	)
+	(text "Warystor przed bezpiecznikiem?"
+		(exclude_from_sim no)
+		(at 91.186 69.342 0)
+		(effects
+			(font
+				(size 1.27 1.27)
+			)
+		)
+	)
+	(text "Sprawdzić opór bezpiecznika resetowalnego"
+		(exclude_from_sim no)
+		(at 179.07 77.47 0)
+		(effects
+			(font
+				(size 1.27 1.27)
+			)
 		)
 	)
