File: kicad/psu_9vdc.kicad_sch (KiCad schematic)
At the start: 5 parts, among them U1 LM7809_TO220

Commit message: Post zip cleanups
Parts:
- added C5, C6: 470u, cap-470u:ESH_13X20_, symbol Device:C_Polarized
- added C7: 330u, cap-330u:CAPPRD500W60D1000H2200, symbol Device:C_Polarized
- C10: footprint (none) -> cap-33u:EEE0JA152UAP
- C8: value 0.33u -> 0.1u; footprint (none) -> Capacitor_SMD:C_0805_2012Metric
- C9: value 100n -> 0.1u; footprint (none) -> Capacitor_SMD:C_0805_2012Metric
- D2: footprint (none) -> Diode_SMD:D_SOD-523
Connections:
- net +12VDC: now also C5.1, C6.1, C7.1
- net GND: now also C5.2, C6.2, C7.2
Other:
- moved on the sheet: C10, C8, C9, D2

Commit message: Initial PCB layout
Parts:
- added D2: D, diode:SE8D20DHM3H, symbol Device:D
- renumbered D2 to D3
Connections:
- net +12VDC: now also D2.1 (K)
- net +9VDC: now also D2.2 (A)
Changed lines of the file:
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@@
+	(wire
+		(pts
+			(xy 152.4 78.74) (xy 157.48 78.74)
+		)
+		(stroke
+			(width 0)
+			(type default)
+		)
+	)
 	(wire
 		(pts
@@
 	(wire
 		(pts
+			(xy 144.78 78.74) (xy 138.43 78.74)
+		)
+		(stroke
+			(width 0)
+			(type default)
+		)
+	)
+	(wire
+		(pts
 			(xy 148.59 96.52) (xy 148.59 99.06)
 		)
@@
 	(wire
 		(pts
+			(xy 138.43 78.74) (xy 138.43 88.9)
+		)
+		(stroke
+			(width 0)
+			(type default)
+		)
+	)
+	(wire
+		(pts
 			(xy 115.57 88.9) (xy 123.19 88.9)
 		)
@@
 		(pts
 			(xy 156.21 88.9) (xy 157.48 88.9)
+		)
+		(stroke
+			(width 0)
+			(type default)
+		)
+	)
+	(wire
+		(pts
+			(xy 157.48 78.74) (xy 157.48 88.9)
 		)
 		(stroke
@@
 		(dnp no)
 		(fields_autoplaced yes)
-		(property "Reference" "D2"
+		(property "Reference" "D3"
 			(at 175.26 92.7099 90)
 			(effects
@@
 			(project "sk"
 				(path "/87c8109f-f49d-4ab5-a5ef-17a7399b7634/efa4e69a-4614-448a-9831-4ab9a658b588"
-					(reference "D2")
+					(reference "D3")
 					(unit 1)
 				)
 				(path "/87c8109f-f49d-4ab5-a5ef-17a7399b7634/dcce0706-074c-494e-9b26-947f484c3154"
-					(reference "D3")
+					(reference "D5")
 					(unit 1)
 				)
 				(path "/87c8109f-f49d-4ab5-a5ef-17a7399b7634/5d1ecf35-531b-475d-b9e1-ef019c8b1c41"
-					(reference "D4")
+					(reference "D7")
 					(unit 1)
 				)
 				(path "/87c8109f-f49d-4ab5-a5ef-17a7399b7634/8149df77-7da5-41c7-bb3d-613defbb0ee6"
-					(reference "D5")
+					(reference "D9")
 					(unit 1)
 				)
 				(path "/87c8109f-f49d-4ab5-a5ef-17a7399b7634/b6273c7b-bd40-4ea1-9f88-7ee3b3d77c26"
-					(reference "D6")
+					(reference "D11")
 					(unit 1)
 				)
 				(path "/87c8109f-f49d-4ab5-a5ef-17a7399b7634/b64cff26-7283-4fb8-a4b0-f105d3ea1cb5"
-					(reference "D7")
+					(reference "D13")
 					(unit 1)
 				)
@@
 		(on_board yes)
 		(dnp no)
-		(property "Reference" "#PWR03"
+		(property "Reference" "#PWR09"
 			(at 148.59 105.41 0)
 			(effects
@@
 			(project "sk"
 				(path "/87c8109f-f49d-4ab5-a5ef-17a7399b7634/efa4e69a-4614-448a-9831-4ab9a658b588"
-					(reference "#PWR03")
+					(reference "#PWR09")
 					(unit 1)
 				)
 				(path "/87c8109f-f49d-4ab5-a5ef-17a7399b7634/dcce0706-074c-494e-9b26-947f484c3154"
-					(reference "#PWR04")
+					(reference "#PWR010")
 					(unit 1)
 				)
 				(path "/87c8109f-f49d-4ab5-a5ef-17a7399b7634/5d1ecf35-531b-475d-b9e1-ef019c8b1c41"
-					(reference "#PWR05")
+					(reference "#PWR011")
 					(unit 1)
 				)
 				(path "/87c8109f-f49d-4ab5-a5ef-17a7399b7634/8149df77-7da5-41c7-bb3d-613defbb0ee6"
-					(reference "#PWR06")
+					(reference "#PWR012")
 					(unit 1)
 				)
 				(path "/87c8109f-f49d-4ab5-a5ef-17a7399b7634/b6273c7b-bd40-4ea1-9f88-7ee3b3d77c26"
-					(reference "#PWR07")
+					(reference "#PWR013")
 					(unit 1)
 				)
 				(path "/87c8109f-f49d-4ab5-a5ef-17a7399b7634/b64cff26-7283-4fb8-a4b0-f105d3ea1cb5"
-					(reference "#PWR08")
+					(reference "#PWR014")
 					(unit 1)
 				)
@@
 					(unit 1)
 				)
+			)
+		)
+	)
+	(symbol
+		(lib_id "Device:D")
+		(at 148.59 78.74 0)
+		(unit 1)
+		(exclude_from_sim no)
+		(in_bom yes)
+		(on_board yes)
+		(dnp no)
+		(property "Reference" "D2"
+			(at 148.59 73.406 0)
+			(effects
+				(font
+					(size 1.27 1.27)
+				)
+			)
+		)
+		(property "Value" "D"
+			(at 148.59 75.692 0)
+			(effects
+				(font
+					(size 1.27 1.27)
+				)
+			)
+		)
+		(property "Footprint" "diode:SE8D20DHM3H"
+			(at 148.59 78.74 0)
+			(effects
+				(font
+					(size 1.27 1.27)
+				)
+				(hide yes)
+			)
+		)
+		(property "Datasheet" "~"
+			(at 148.59 78.74 0)
+			(effects
+				(font
+					(size 1.27 1.27)
+				)
+				(hide yes)
+			)
+		)
+		(property "Description" "Diode"
+			(at 148.59 78.74 0)
+			(effects
+				(font
+					(size 1.27 1.27)
+				)
+				(hide yes)
+			)
+		)
+		(property "Sim.Device" "D"
+			(at 148.59 78.74 0)
+			(effects
+				(font
+					(size 1.27 1.27)
+				)
+				(hide yes)
+			)
+		)
+		(property "Sim.Pins" "1=K 2=A"
+			(at 148.59 78.74 0)
+			(effects
+				(font
+					(size 1.27 1.27)
+				)
+				(hide yes)
+			)
+		)
+		(pin "2"
+		)
+		(pin "1"
+		)
+		(instances
+			(project "sk"
+				(path "/87c8109f-f49d-4ab5-a5ef-17a7399b7634/efa4e69a-4614-448a-9831-4ab9a658b588"
+					(reference "D2")
+					(unit 1)
+				)
+				(path "/87c8109f-f49d-4ab5-a5ef-17a7399b7634/dcce0706-074c-494e-9b26-947f484c3154"
+					(reference "D4")
+					(unit 1)
+				)
+				(path "/87c8109f-f49d-4ab5-a5ef-17a7399b7634/5d1ecf35-531b-475d-b9e1-ef019c8b1c41"
+					(reference "D6")
+					(unit 1)
+				)
+				(path "/87c8109f-f49d-4ab5-a5ef-17a7399b7634/8149df77-7da5-41c7-bb3d-613defbb0ee6"
+					(reference "D8")
+					(unit 1)
+				)
+				(path "/87c8109f-f49d-4ab5-a5ef-17a7399b7634/b6273c7b-bd40-4ea1-9f88-7ee3b3d77c26"
+					(reference "D10")
+					(unit 1)
+				)
+				(path "/87c8109f-f49d-4ab5-a5ef-17a7399b7634/b64cff26-7283-4fb8-a4b0-f105d3ea1cb5"
+					(reference "D12")
+					(unit 1)
+				)

Commit message: Make PCB rework
Parts:
- added D2: LED, Diode_SMD:D_0805_2012Metric, symbol Device:LED
- added R1: 680, Resistor_SMD:R_0805_2012Metric, symbol Device:R
- added SW1: SW_DIP_x01, switch:200MSP1T1B1M2QEH, symbol Switch:SW_DIP_x01
- renumbered D2 to D3, D3 to D4
Connections:
- net +12VDC: now also SW1.1; no longer C8.1, D3.1 (K), U1.1 (VI)
- net GND: now also D2.2 (A)
- new net: C8.1, D3.1 (K), R1.1, SW1.2, U1.1 (VI)
- new net: D2.1 (K), R1.2
Other:
- moved on the sheet: C10, C8, C9, D3, D4, U1

Commit message: Post review
Connections:
- net GND: now also D2.1 (K); no longer D2.2 (A)
- net at R1.2: now also D2.2 (A); no longer D2.1 (K)
Other:
- moved on the sheet: D2
Changed lines of the file:
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@@
+	)
+	(junction
+		(at 109.22 115.57)
+		(diameter 0)
+		(color 0 0 0 0)
 	)
 	(junction
@@
 	)
 	(junction
-		(at 109.22 114.3)
-		(diameter 0)
-		(color 0 0 0 0)
-	)
-	(junction
 		(at 109.22 99.06)
 		(diameter 0)
@@
 	(wire
 		(pts
-			(xy 91.44 109.22) (xy 91.44 114.3)
+			(xy 91.44 109.22) (xy 91.44 115.57)
 		)
 		(stroke
@@
 	(wire
 		(pts
+			(xy 109.22 115.57) (xy 109.22 114.3)
+		)
+		(stroke
+			(width 0)
+			(type default)
+		)
+	)
+	(wire
+		(pts
 			(xy 138.43 109.22) (xy 138.43 107.95)
 		)
@@
 	(wire
 		(pts
-			(xy 119.38 114.3) (xy 119.38 109.22)
+			(xy 119.38 115.57) (xy 119.38 109.22)
 		)
 		(stroke
@@
 	(wire
 		(pts
+			(xy 109.22 115.57) (xy 119.38 115.57)
+		)
+		(stroke
+			(width 0)
+			(type default)
+		)
+	)
+	(wire
+		(pts
 			(xy 138.43 99.06) (xy 146.05 99.06)
 		)
@@
 	(wire
 		(pts
-			(xy 91.44 114.3) (xy 109.22 114.3)
+			(xy 91.44 115.57) (xy 109.22 115.57)
 		)
 		(stroke
@@
 		(pts
 			(xy 153.67 99.06) (xy 161.29 99.06)
-		)
-		(stroke
-			(width 0)
-			(type default)
-		)
-	)
-	(wire
-		(pts
-			(xy 109.22 114.3) (xy 119.38 114.3)
 		)
 		(stroke
@@
 	(symbol
 		(lib_id "Device:LED")
-		(at 109.22 110.49 270)
+		(at 109.22 110.49 90)
 		(unit 1)
 		(exclude_from_sim no)
@@
 		(fields_autoplaced yes)
 		(property "Reference" "D2"
-			(at 111.76 107.6324 90)
-			(effects
-				(font
-					(size 1.27 1.27)
-				)
-				(justify left)
+			(at 113.03 110.8074 90)
+			(effects
+				(font
+					(size 1.27 1.27)
+				)
+				(justify right)
 			)
 		)
 		(property "Value" "LED"
-			(at 111.76 110.1724 90)
-			(effects
-				(font
-					(size 1.27 1.27)
-				)
-				(justify left)
-			)
-		)
+			(at 113.03 113.3474 90)
+			(effects
+				(font
+					(size 1.27 1.27)
+				)
+				(justify right)
+			)
+		)
